File: EcoJM/EcoJM.kicad_sch (KiCad schematic)
At the start: 50 parts, among them J1 Conn_01x01_Pin, J10 Conn_01x01_Pin, J11 Conn_01x01_Pin, J2 Conn_01x01_Pin, J3 Conn_01x02_Pin, J4 Conn_01x02_Pin, J5 Conn_01x03_Pin, J6 Conn_01x02_Pin, J7 Conn_01x03_Pin, J8 Screw_Terminal_01x02, J9 Screw_Terminal_01x02, Q1 2SD882_C842818, Q2 2SD882_C842818, U1 ACS712xLCTR-30A, U2 MT2492, U3 SIT65HVD230DR, U4 AZ1117-3.3, U5 RS321BXF, U6 STM32F_dev, U7 PC817C_C3025164, U8 PC817C_C3025164

Commit message: update
Parts:
- J1, J10, J11, J2: footprint (none) -> Connector_Wire:SolderWirePad_1x01_SMD_5x10mm
Connections:
- net SSR0: now also U6.13 (B5); no longer U6.28 (B0)
- net SSR1: now also U6.12 (B4); no longer U6.27 (B1)
Changed lines of the file:
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@@
 		)
 	)
+	(text_box "PSU"
+		(exclude_from_sim no)
+		(at 13.97 138.43 0)
+		(size 153.67 58.42)
+		(margins 0.9525 0.9525 0.9525 0.9525)
+		(stroke
+			(width 0)
+			(type solid)
+		)
+		(fill
+			(type none)
+		)
+		(effects
+			(font
+				(size 1.27 1.27)
+			)
+			(justify left top)
+		)
+	)
 	(junction
 		(at 118.11 162.56)
@@
 	)
 	(no_connect
-		(at 29.21 85.09)
+		(at 64.77 85.09)
 	)
 	(no_connect
-		(at 29.21 100.33)
+		(at 29.21 85.09)
 	)
 	(no_connect
@@
 	)
 	(no_connect
-		(at 29.21 62.23)
+		(at 64.77 81.28)
 	)
 	(no_connect
-		(at 29.21 88.9)
+		(at 29.21 62.23)
 	)
 	(no_connect
-		(at 29.21 104.14)
+		(at 29.21 88.9)
 	)
 	(no_connect
@@
 	(wire
 		(pts
-			(xy 64.77 85.09) (xy 66.04 85.09)
-		)
-		(stroke
-			(width 0)
-			(type default)
-		)
-	)
-	(wire
-		(pts
 			(xy 214.63 100.33) (xy 214.63 102.87)
 		)
@@
 	(wire
 		(pts
+			(xy 27.94 104.14) (xy 29.21 104.14)
+		)
+		(stroke
+			(width 0)
+			(type default)
+		)
+	)
+	(wire
+		(pts
 			(xy 60.96 46.99) (xy 66.04 46.99)
 		)
@@
 	(wire
 		(pts
-			(xy 64.77 81.28) (xy 66.04 81.28)
+			(xy 27.94 100.33) (xy 29.21 100.33)
 		)
 		(stroke
@@
 		)
 	)
-	(label "SSR0"
-		(at 66.04 85.09 0)
+	(label "SSR1"
+		(at 27.94 100.33 180)
 		(effects
 			(font
 				(size 1.27 1.27)
 			)
-			(justify left bottom)
+			(justify right bottom)
 		)
 	)
@@
 		)
 	)
-	(label "SSR1"
-		(at 66.04 81.28 0)
-		(effects
-			(font
-				(size 1.27 1.27)
-			)
-			(justify left bottom)
-		)
-	)
 	(label "CAN_RXD"
 		(at 20.32 115.57 0)
@@
 		)
 	)
+	(label "SSR0"
+		(at 27.94 104.14 180)
+		(effects
+			(font
+				(size 1.27 1.27)
+			)
+			(justify right bottom)
+		)
+	)
 	(symbol
 		(lib_id "power:GND")
@@
 			)
 		)
-		(property "Footprint" ""
+		(property "Footprint" "Connector_Wire:SolderWirePad_1x01_SMD_5x10mm"
 			(at 264.16 139.7 0)
 			(effects
@@
 		(on_board yes)
 		(dnp no)
-		(fields_autoplaced yes)
 		(property "Reference" "J2"
 			(at 239.395 130.81 0)
@@
 		)
 		(property "Value" "Conn_01x01_Pin"
-			(at 239.395 133.35 0)
+			(at 239.268 137.414 0)
 			(effects
 				(font
@@
 			)
 		)
-		(property "Footprint" ""
+		(property "Footprint" "Connector_Wire:SolderWirePad_1x01_SMD_5x10mm"
 			(at 240.03 135.89 0)
 			(effects
@@
 			)
 		)
-		(property "Footprint" ""
+		(property "Footprint" "Connector_Wire:SolderWirePad_1x01_SMD_5x10mm"
 			(at 240.03 133.35 0)
 			(effects
@@
 		)
 		(property "Value" "Conn_01x01_Pin"
-			(at 264.795 139.7 0)
+			(at 264.16 144.272 0)
 			(effects
 				(font
@@
 			)
 		)
-		(property "Footprint" ""
+		(property "Footprint" "Connector_Wire:SolderWirePad_1x01_SMD_5x10mm"
 			(at 264.16 142.24 0)
 			(effects
