File: EcoJM/EcoJM.kicad_sch (KiCad schematic)
At the start: 43 parts, among them J1 Conn_01x01_Pin, J10 Conn_01x01_Pin, J11 Conn_01x01_Pin, J12 Micro_SD_Card, J2 Conn_01x01_Pin, J3 Conn_01x02_Pin, J4 Conn_01x02_Pin, J5 Conn_01x03_Pin, J6 Conn_01x02_Pin, J7 Conn_01x03_Pin, J8 Screw_Terminal_01x02, J9 Screw_Terminal_01x02, Q1 2SD882_C842818, Q2 2SD882_C842818, U1 ACS712xLCTR-30A, U2 MT2492, U4 AZ1117-3.3, U5 SIT1051T/3, U6 STM32F_dev, U7 PC817C_C3025164, U8 PC817C_C3025164

Commit message: RevA finito, revision, reroute, refurbish
Parts:
- removed C3, C4: 22u, LED_SMD:LED_1206_3216Metric_Pad1.42x1.75mm_HandSolder, symbol Device:C
- removed C6: 22n, LED_SMD:LED_1206_3216Metric_Pad1.42x1.75mm_HandSolder, symbol Device:C
- removed F1: Fuse, Fuse:Fuseholder_Clip-5x20mm_Keystone_3512_Inline_P23.62x7.27mm_D1.02x1.57mm_Horizontal, symbol Device:Fuse
- removed J1, J10, J11, J2: Conn_01x01_Pin, Connector_Wire:SolderWirePad_1x01_SMD_5x10mm, symbol Connector:Conn_01x01_Pin
- removed J12: Micro_SD_Card, symbol Connector:Micro_SD_Card
- removed J4, J6: Conn_01x02_Pin, Connector_PinHeader_2.54mm:PinHeader_1x02_P2.54mm_Vertical, symbol Connector:Conn_01x02_Pin
- removed J5, J7: Conn_01x03_Pin, Connector_JST:JST_XH_B3B-XH-A_1x03_P2.50mm_Vertical, symbol Connector:Conn_01x03_Pin
- removed J8, J9: Screw_Terminal_01x02, TerminalBlock_Phoenix:TerminalBlock_Phoenix_PT-1,5-2-3.5-H_1x02_P3.50mm_Horizontal, symbol Connector:Screw_Terminal_01x02
- removed L1: 10u, EasyEDA:IND-SMD_L7.2-W6.6_GPSR07X0, symbol Device:L
- removed Q1, Q2: 2SD882_C842818, EasyEDA:SOT-89-3_L4.5-W2.5-P1.50-LS4.1-BR, symbol EasyEDA:2SD882_C842818
- removed R1, R2: 10k, Resistor_SMD:R_1206_3216Metric_Pad1.30x1.75mm_HandSolder, symbol Device:R
- removed R13, R8: 470, Resistor_SMD:R_1206_3216Metric_Pad1.30x1.75mm_HandSolder, symbol Device:R
- removed R14, R15: 100, Resistor_SMD:R_1206_3216Metric_Pad1.30x1.75mm_HandSolder, symbol Device:R
- removed R3: 110k, Resistor_SMD:R_1206_3216Metric_Pad1.30x1.75mm_HandSolder, symbol Device:R
- removed R4: 15k, Resistor_SMD:R_1206_3216Metric_Pad1.30x1.75mm_HandSolder, symbol Device:R
- removed R5: 120, Resistor_SMD:R_1206_3216Metric_Pad1.30x1.75mm_HandSolder, symbol Device:R
- removed TP1, TP2: TestPoint, TestPoint:TestPoint_Pad_D1.5mm, symbol Connector:TestPoint
- removed U2: MT2492, EasyEDA:SOT-23-6_L2.9-W1.6-P0.95-LS2.8-BL_3, symbol EasyEDA:MT2492
- removed U5: SIT1051T/3, EasyEDA:SOP-8_L4.9-W3.9-P1.27-LS6.0-BL, symbol EasyEDAA:SIT1051T_3
- removed U7, U8: PC817C_C3025164, EasyEDA:OPTO-SMD-4_L4.6-W6.5-P2.54-LS10.3-TL, symbol EasyEDA:PC817C_C3025164
- added C10: 10u, Capacitor_SMD:C_1206_3216Metric_Pad1.33x1.80mm_HandSolder, symbol Device:C
- added C11: 22u, Capacitor_SMD:C_1206_3216Metric_Pad1.33x1.80mm_HandSolder, symbol Device:C
- added C8: 1u, Capacitor_SMD:C_0603_1608Metric_Pad1.08x0.95mm_HandSolder, symbol Device:C
- added C9: 22n, Capacitor_SMD:C_0603_1608Metric_Pad1.08x0.95mm_HandSolder, symbol Device:C
- added D1: P6KE47A, Diode_THT:D_DO-15_P10.16mm_Horizontal, symbol Device:D_Unitunnel
- added D2: SS14, Diode_SMD:D_SMA, symbol Diode:SS14
- added F2: Fuse, Fuse:Fuseholder_Clip-5x20mm_Littelfuse_520_Inline_P20.50x5.80mm_D1.30mm_Horizontal, symbol Device:Fuse
- added H1, H2, H3, H4: MountingHole, MountingHole:MountingHole_3.2mm_M3_DIN965, symbol Mechanical:MountingHole
- added J1: Screw_Terminal_01x02, TerminalBlock_Phoenix:TerminalBlock_Phoenix_MKDS-1,5-2_1x02_P5.00mm_Horizontal, symbol Connector:Screw_Terminal_01x02
- added J10, J5: Conn_01x02_Pin, Connector_PinHeader_2.54mm:PinHeader_1x02_P2.54mm_Vertical, symbol Connector:Conn_01x02_Pin
- added J4: Conn_01x04_Pin, Connector_JST:JST_XH_B4B-XH-A_1x04_P2.50mm_Vertical, symbol Connector:Conn_01x04_Pin
- added J6, J7, J8, J9: Screw_Terminal_01x01, Libmain:M3_PCONN_1x01, symbol Connector:Screw_Terminal_01x01
- added K1: Relay_SPDT, liblocal:T91 30A, symbol Relay:Relay_SPDT
- added L2: CD54-6R8M, EasyEDA:IND-SMD_L5.8-W5.2_CD54, symbol EasyEDA:CD54-150M_C49230812
- added Q1: AO3400A, Package_TO_SOT_SMD:SOT-23, symbol Transistor_FET:AO3400A
- added R10: 2.7k, Resistor_SMD:R_1206_3216Metric_Pad1.30x1.75mm_HandSolder, symbol Device:R
- added R11: 10k, Capacitor_SMD:C_0603_1608Metric_Pad1.08x0.95mm_HandSolder, symbol Device:R
- added R12: 120, Resistor_SMD:R_1206_3216Metric_Pad1.30x1.75mm_HandSolder, symbol Device:R
- added R16: 110k, Resistor_SMD:R_0603_1608Metric_Pad0.98x0.95mm_HandSolder, symbol Device:R
- added R17: 15k, Resistor_SMD:R_0603_1608Metric_Pad0.98x0.95mm_HandSolder, symbol Device:R
- added R18: 10k, Resistor_SMD:R_0603_1608Metric_Pad0.98x0.95mm_HandSolder, symbol Device:R
- added R19: 470, Resistor_SMD:R_0603_1608Metric_Pad0.98x0.95mm_HandSolder, symbol Device:R
- added R20: 2k, Resistor_SMD:R_0603_1608Metric_Pad0.98x0.95mm_HandSolder, symbol Device:R
- added R21: 20k, Resistor_SMD:R_0603_1608Metric_Pad0.98x0.95mm_HandSolder, symbol Device:R
- added R9: 47k, Resistor_SMD:R_1206_3216Metric_Pad1.30x1.75mm_HandSolder, symbol Device:R
- added U10: MT2492, EasyEDA:SOT-23-6_L2.9-W1.6-P0.95-LS2.8-BL_3, symbol EasyEDA:MT2492
- added U2: TL431DBZ, Package_TO_SOT_SMD:SOT-23, symbol Reference_Voltage:TL431DBZ
- added U5: HX TF PUSH, EasyEDA:TF-SMD_TF-PUSH, symbol EasyEDA:HXTFPUSH
- added U9: SIT65HVD230DR, EasyEDA:SOP-8_L4.9-W3.9-P1.27-LS6.0-BL, symbol EasyEDA:SIT65HVD230DR
- C1, C2, C5: footprint LED_SMD:LED_1206_3216Metric_Pad1.42x1.75mm_HandSolder -> Capacitor_SMD:C_0603_1608Metric_Pad1.08x0.95mm_HandSolder
- C7: footprint LED_SMD:LED_1206_3216Metric_Pad1.42x1.75mm_HandSolder -> Capacitor_SMD:C_1206_3216Metric_Pad1.33x1.80mm_HandSolder
- R6, R7: footprint Resistor_SMD:R_1206_3216Metric_Pad1.30x1.75mm_HandSolder -> Capacitor_SMD:C_0603_1608Metric_Pad1.08x0.95mm_HandSolder
Connections:
- net +12V: now also C10.1, D2.1 (K), K1.A1, R18.1, U10.5 (IN)
- net +3.3V: now also C5.1, C8.1, R19.1, U5.4 (VDD), U9.3 (VCC); no longer C5.2
- net +5V: now also C11.1, L2.2, R16.1
- net CAN_RXD: now also U9.4 (R)
- net CAN_TXD: now also U9.1 (D)
- net GND: now also C5.2, C10.2, C11.2, C8.2, J10.2 (Pin_2), J4.3 (Pin_3), J4.4 (Pin_4), Q1.2 (S), R10.2, R11.1, R17.2, R21.1, U10.2 (GND), U2.3 (A), U5.10 (SHELL), U5.11 (SHELL), U5.12 (SHELL), U5.13 (SHELL), U5.6 (VSS), U9.2 (GND); no longer C5.1
- net SD_CS: now also U5.2 (CD/DAT3)
- net SPI_MISO: now also U5.7 (DAT0)
- net SPI_MOSI: now also U5.3 (CMD)
- net SPI_SCK: now also U5.5 (CLK)
- net SSR0: now also R20.2
- net VDCH+_IN: now also J6.1 (Pin_1), K1.14
- net VDCH+_OUT: now also J8.1 (Pin_1)
- net VDCH-: now also D1.2 (A), J7.1 (Pin_1), J9.1 (Pin_1)
- net Voltage_M: now also R10.1, R9.1
- net VREF: now reaches U6.34 (A2)
- net VREF: now also R19.2, U2.1 (K), U2.2 (REF)
- net VDCH+_INFUSED: now reaches U1.1 (IP+), U1.2 (IP+)
- net VDCH+_INFUSED: now also D1.1 (K), F2.2, R9.2
- net SSR1: no longer names the net of U6.12 (B4)
- net UART_RX: no longer names the net of U6.15 (B7)
- net UART_TX: no longer names the net of U6.14 (B6)
- new net: J1.1 (Pin_1), J10.1 (Pin_1), Q1.3 (D)
- new net: D2.2 (A), J1.2 (Pin_2), K1.A2
- new net: R11.2, U9.8 (RS)
- new net: C9.1, L2.1, U10.6 (SW)
- new net: R16.2, R17.1, U10.3 (FB)
- new net: Q1.1 (G), R20.1, R21.2
- new net: J5.2 (Pin_2), R12.2
- new net: C9.2, U10.1 (BS)
- new net: R18.2, U10.4 (EN)
- new net CANH: J4.1 (Pin_1), J5.1 (Pin_1), U9.7 (CANH)
- new net CANL: J4.2 (Pin_2), R12.1, U9.6 (CANL)
- new net VDCH+_INSW: F2.1, K1.11
- no-connect marks 28 -> 31
Other:
- moved on the sheet: C1, C7, J3, U4, U6

Commit message: Quick fix, minor modifications
Parts:
- added J11, J12: Screw_Terminal_01x01, Connector_Wire:SolderWire-0.25sqmm_1x01_D0.65mm_OD1.7mm_Relief, symbol Connector:Screw_Terminal_01x01
Connections:
- net +3.3V: now also R21.2
- net GND: no longer R21.1
- net VDCH+_IN: now also U1.3 (IP-), U1.4 (IP-); no longer K1.14
- net VDCH+_INFUSED: no longer D1.1 (K)
- net VDCH+_INSW: now also J12.1 (Pin_1)
- net VDCH+_OUT: now also D1.1 (K), K1.14; no longer U1.3 (IP-), U1.4 (IP-)
- net VDCH-: now also J11.1 (Pin_1)
- net at Q1.1 (G), R20.1: now also R21.1; no longer R21.2
Other:
- moved on the sheet: J6, J8, R21
